File: Hardware/KiCad/Grape/usb_communication.sch (KiCad schematic (older format))
At the start: 8 parts

Commit message: Primera pagina terminada
Parts:
- removed C?: C_Small, symbol C_Small
- removed U?: FT231XS, SSOP-20, symbol FT231XS
- removed X?: USB-MB-S, miniusb, symbol USB-MB-S
- added C1, C2, C4: 0.1uF, symbol C_Small
- added C19, C20: 47pF, symbol C_Small
- added D2: GREEN, symbol LED_Small_ALT
- added J1: USB_MICROB, USB-B-MICRO-SMD_V03, symbol USB_MICROB_PLUGCONN-11752
- added R1, R4, R5, R6: 1k, symbol R_Small
- added R13: 27R, symbol R_Small
- added R14, R15: 10k, symbol R_Small
- added U1: FT231XS, SSOP-20, symbol FT231XS
- C3: renamed from C?; value CP1_Small -> CP1_SmalluF
- D1: renamed from D?; value LED_Small_ALT -> RED
- F2: renamed from F?; value Polyfuse_Small -> 500mA
- Q1: renamed from Q?; value MOSFET-NCHANNEL2N7002PW -> 2N7002PW
- R12: renamed from R?; value R_Small -> 27R
Connections:
- net labels added: +3.3V, +5V, DTR, GND, RX, TX, USB_5V
- wire segments 0 -> 64
- no-connect marks 0 -> 8
Other:
- moved on the sheet: C3, D1, F2, Q1, R12
