File: Hardware/KiCad/Grape/Power.sch (KiCad schematic (older format))
At the start: 0 parts

Commit message: Alimentacion comenzada
Parts:
- added D?: MBRA140, SMA-DIODE, symbol MBRA140
- added J?: POWER_JACKPTH, POWER_JACK_PTH, symbol POWER_JACKPTH
- added SW?: SW_SPDT, symbol SW_SPDT
Connections:
- new net: J?.PWR, SW?.2 (B)
- new net: D?.A, SW?.1 (A)
- new net GND: J?.GND, J?.GNDB (GNDBREAK)
Changed lines of the file:
@@
 $Descr A4 11693 8268
 encoding utf-8
-Sheet 1 5
+Sheet 5 5
 Title ""
 Date ""
@@
 Comment4 ""
 $EndDescr
+$Comp
+L POWER_JACKPTH J?
+U 1 1 5A5C9961
+P 3400 2950
+F 0 "J?" H 3000 2950 50  0000 L BNN
+F 1 "POWER_JACKPTH" H 3000 3350 50  0000 L BNN
+F 2 "POWER_JACK_PTH" H 3430 3100 20  0001 C CNN
+F 3 "" H 3400 2950 60  0000 C CNN
+	1    3400 2950
+	1    0    0    -1
+$EndComp
+$Comp
+L MBRA140 D?
+U 1 1 5A5C99D2
+P 4450 2650
+F 0 "D?" H 4550 2669 50  0000 L BNN
+F 1 "MBRA140" H 4550 2559 50  0000 L BNN
+F 2 "SMA-DIODE" H 4480 2800 20  0001 C CNN
+F 3 "" H 4450 2650 60  0001 C CNN
+	1    4450 2650
+	1    0    0    -1
+$EndComp
+$Comp
+L SW_SPDT SW?
+U 1 1 5A5C9A3B
+P 3950 2650
+F 0 "SW?" H 3950 2820 50  0000 C CNN
+F 1 "SW_SPDT" H 3950 2450 50  0000 C CNN
+F 2 "" H 3950 2650 50  0001 C CNN
+F 3 "" H 3950 2650 50  0001 C CNN
+	1    3950 2650
+	1    0    0    -1
+$EndComp
+Wire Wire Line
+	3500 2650 3750 2650
+Wire Wire Line
+	4150 2550 4250 2550
+Wire Wire Line
+	4250 2550 4250 2650
+Wire Wire Line
+	4250 2650 4350 2650
+$Comp
+L GND #PWR?
+U 1 1 5A5C9A9A
+P 3650 3050
+F 0 "#PWR?" H 3650 2800 50  0001 C CNN
+F 1 "GND" H 3650 2900 50  0000 C CNN
+F 2 "" H 3650 3050 60  0000 C CNN
+F 3 "" H 3650 3050 60  0000 C CNN
+	1    3650 3050
+	1    0    0    -1
+$EndComp
+Wire Wire Line
+	3500 2750 3650 2750
+Wire Wire Line
+	3650 2750 3650 3050
+Wire Wire Line
+	3500 2850 3650 2850
+Connection ~ 3650 2850
 $EndSCHEMATC

Commit message: Alimentacion terminada
Parts:
- added C10, C11, C22, C23, C24: 100nF, symbol C_Small
- added C15: 100n, symbol C_Small
- added C16: 10n, symbol C_Small
- added C7: 100u, symbol CP1_Small
- added C8: 3.3n, symbol C_Small
- added C9: 100uF, symbol CP1_Small
- added L1: 10uH, symbol L_Small
- added L2: 60R 100M Ferrite, symbol L_Small
- added Q4, Q5: FDN340P, SOT23-3, symbol MOSFET-PCHANNEL
- added R10: 1k 1%, symbol R_Small
- added R11: 100k, symbol R_Small
- added R16, R17, R18, R20: 10k, symbol R_Small
- added R7: 5K6 1%, symbol R_Small
- added R9: 6.8k, symbol R_Small
- added U2: LM358, symbol LM358
- added U3: AMS1117-3.3, SOT223, symbol V_REG_LM1117SOT223
- added U8: MP2307SO, symbol MP2307SO
- gave numbers to parts that had none: 3
Connections:
- net GND: now also C10.2, C11.2, C15.2, C22.2, C23.2, C24.2, C7.2, C9.2, R10.1, R17.1, R9.2, U2.4 (V-), U2.4 (V-), U3.1 (ADJ), U8.4 (GND), U8.9 (GND_TP)
- net VIN: now reaches D5.C
- net VIN: now also C10.1, C9.1, R11.2, R18.2, U8.2 (IN)
- new net: C16.2, U8.1 (BS)
- new net: C16.1, L1.1, U8.3 (SW)
- new net: R10.2, R7.1, U8.5 (FB)
- new net: C8.1, U8.6 (COMP)
- new net: R11.1, U8.7 (EN)
- new net: C11.1, U8.8 (SS)
- new net: C8.2, R9.1
- new net: C15.1, C7.1, L1.2, L2.1, R7.2
- new net: Q4.1 (G), R20.1, U2.1
- new net: C22.1, R17.2, R18.1, U2.3 (+), U2.6 (-)
- new net: Q5.1 (G), R16.1, U2.7
- new net +3V3: C24.1, U2.2 (-), U2.5 (+), U3.2 (OUT), U3.4 (OUT)
- new net +5V: C23.1, Q4.2 (S), Q5.2 (S), R16.2, R20.2, U2.8 (V+), U2.8 (V+), U3.3 (IN)
- new net USB_5V: Q4.3 (D)
- new net VDD5: L2.2, Q5.3 (D)
- no-connect marks 0 -> 1
Other:
- moved on the sheet: D5, J19, SW1

Commit message: Esquema terminado y  ERC pasado
Other:
- note added: "3V LDO"
- note added: "Step-Down Converter"
- note added: "USB Auto-Selector"
- moved on the sheet: C10, C11, C15, C16, C22, C23, C24, C7, C8, C9, D5, J19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

Commit message: cvpcb terminado
Parts:
- C10, C11, C15, C16, C22, C23, C24, C8: footprint (none) -> Capacitors_SMD:C_0805
- C7, C9: footprint (none) -> Capacitors_SMD:CP_Elec_6.3x5.3
- D1: renamed from D5; footprint SMA-DIODE -> Diodes_SMD:D_SMA
- J19: footprint POWER_JACK_PTH -> Connectors:JACK_ALIM
- L1: footprint (none) -> Inductors_SMD:L_Wuerth_WE-PD2-Typ-L
- L2: footprint (none) -> Inductors_SMD:L_0805
- Q4, Q5: footprint SOT23-3 -> TO_SOT_Packages_SMD:SOT-23
- R10, R11, R16, R17, R18, R20, R7, R9: footprint (none) -> Resistors_SMD:R_0805
- SW1: footprint (none) -> Buttons_Switches_SMD:SW_SPDT_PCM12
- U2: footprint (none) -> Housings_SOIC:SOIC-8_3.9x4.9mm_Pitch1.27mm
- U3: footprint SOT223 -> TO_SOT_Packages_SMD:SOT-223
- U8: footprint (none) -> Housings_SOIC:HTSOP-8-1EP_3.9x4.9mm_Pitch1.27mm_ThermalVias_LargeCopper
Changed lines of the file:
@@
 F 0 "J19" H 2500 2550 50  0000 L BNN
 F 1 "POWER_JACKPTH" H 2500 2950 50  0000 L BNN
-F 2 "POWER_JACK_PTH" H 2930 2700 20  0001 C CNN
+F 2 "Connectors:JACK_ALIM" H 2930 2700 20  0001 C CNN
 F 3 "" H 2900 2550 60  0000 C CNN
 	1    2900 2550
@@
 $EndComp
 $Comp
-L MBRA140 D5
+L MBRA140 D1
 U 1 1 5A5C99D2
 P 3950 2250
-F 0 "D5" H 3900 2350 50  0000 L BNN
+F 0 "D1" H 3900 2350 50  0000 L BNN
 F 1 "MBRA140" H 3800 2100 50  0000 L BNN
-F 2 "SMA-DIODE" H 3980 2400 20  0001 C CNN
+F 2 "Diodes_SMD:D_SMA" H 3980 2400 20  0001 C CNN
 F 3 "" H 3950 2250 60  0001 C CNN
 	1    3950 2250
@@
 F 0 "SW1" H 3450 2420 50  0000 C CNN
 F 1 "SW_SPDT" H 3450 2050 50  0000 C CNN
-F 2 "" H 3450 2250 50  0001 C CNN
+F 2 "Buttons_Switches_SMD:SW_SPDT_PCM12" H 3450 2250 50  0001 C CNN
 F 3 "" H 3450 2250 50  0001 C CNN
 	1    3450 2250
@@
 F 0 "U8" H 5550 2050 39  0000 C CNN
 F 1 "MP2307SO" H 5900 2550 39  0000 C CNN
-F 2 "" H 5900 2450 39  0001 C CNN
+F 2 "Housings_SOIC:HTSOP-8-1EP_3.9x4.9mm_Pitch1.27mm_ThermalVias_LargeCopper" H 5900 2450 39  0001 C CNN
 F 3 "" H 5900 2450 39  0001 C CNN
 	1    5900 2450
@@
 F 0 "R9" V 6400 2900 50  0000 L CNN
 F 1 "6.8k" V 6600 2900 50  0000 L CNN
-F 2 "" H 6500 2950 50  0001 C CNN
+F 2 "Resistors_SMD:R_0805" H 6500 2950 50  0001 C CNN
 F 3 "" H 6500 2950 50  0001 C CNN
 	1    6500 2950
@@
 F 0 "C8" H 6760 2870 50  0000 L CNN
 F 1 "3.3n" H 6760 2720 50  0000 L CNN
-F 2 "" H 6750 2800 50  0001 C CNN
+F 2 "Capacitors_SMD:C_0805" H 6750 2800 50  0001 C CNN
 F 3 "" H 6750 2800 50  0001 C CNN
 	1    6750 2800
@@
 F 0 "L1" V 7000 2200 50  0000 L CNN
 F 1 "10uH" V 6800 2150 50  0000 L CNN
-F 2 "" H 6900 2250 50  0001 C CNN
+F 2 "Inductors_SMD:L_Wuerth_WE-PD2-Typ-L" H 6900 2250 50  0001 C CNN
 F 3 "" H 6900 2250 50  0001 C CNN
 	1    6900 2250
@@
 F 0 "L2" V 8700 2200 50  0000 L CNN
 F 1 "60R 100M Ferrite" V 8550 2000 39  0000 L CNN
-F 2 "" H 8600 2250 50  0001 C CNN
+F 2 "Inductors_SMD:L_0805" H 8600 2250 50  0001 C CNN
 F 3 "" H 8600 2250 50  0001 C CNN
 	1    8600 2250
@@
 F 0 "U2" H 4200 4950 50  0000 L CNN
 F 1 "LM358" H 4200 4550 50  0000 L CNN
-F 2 "" H 4200 4750 50  0001 C CNN
+F 2 "Housings_SOIC:SOIC-8_3.9x4.9mm_Pitch1.27mm" H 4200 4750 50  0001 C CNN
 F 3 "" H 4200 4750 50  0001 C CNN
 	1    4200 4750
@@
 F 0 "U2" H 4800 5800 50  0000 L CNN
 F 1 "LM358" H 4800 5400 50  0000 L CNN
-F 2 "" H 4800 5600 50  0001 C CNN
+F 2 "Housings_SOIC:SOIC-8_3.9x4.9mm_Pitch1.27mm" H 4800 5600 50  0001 C CNN
 F 3 "" H 4800 5600 50  0001 C CNN
 	2    4800 5600
@@
 F 0 "Q5" V 6000 5450 50  0000 L BNN
 F 1 "FDN340P" V 6000 4750 50  0000 L BNN
-F 2 "SOT23-3" H 6080 5400 20  0001 C CNN
+F 2 "TO_SOT_Packages_SMD:SOT-23" H 6080 5400 20  0001 C CNN
 F 3 "" H 6050 5250 60  0001 C CNN
 	1    6050 5250
@@
 F 0 "U3" H 7800 4200 50  0000 L BNN
 F 1 "AMS1117-3.3" H 7450 4650 50  0000 L BNN
-F 2 "SOT223" H 7730 4650 20  0001 C CNN
+F 2 "TO_SOT_Packages_SMD:SOT-223" H 7730 4650 20  0001 C CNN
 F 3 "" H 7700 4500 60  0001 C CNN
 	1    7700 4500
@@
 F 0 "C9" H 4210 2720 50  0000 L CNN
 F 1 "100uF" H 3950 2550 50  0000 L CNN
-F 2 "" H 4200 2650 50  0001 C CNN
+F 2 "Capacitors_SMD:CP_Elec_6.3x5.3" H 4200 2650 50  0001 C CNN
 F 3 "" H 4200 2650 50  0001 C CNN
 	1    4200 2650
@@
 F 0 "C10" H 4610 2720 50  0000 L CNN
 F 1 "100nF" H 4610 2570 50  0000 L CNN
-F 2 "" H 4600 2650 50  0001 C CNN
+F 2 "Capacitors_SMD:C_0805" H 4600 2650 50  0001 C CNN
 F 3 "" H 4600 2650 50  0001 C CNN
 	1    4600 2650
@@
 F 0 "R11" V 4850 2200 50  0000 L CNN
 F 1 "100k" V 5050 2200 50  0000 L CNN
-F 2 "" H 4950 2250 50  0001 C CNN
+F 2 "Resistors_SMD:R_0805" H 4950 2250 50  0001 C CNN
 F 3 "" H 4950 2250 50  0001 C CNN
 	1    4950 2250
@@
 F 0 "C11" H 5110 2770 50  0000 L CNN
 F 1 "100nF" H 5110 2620 50  0000 L CNN
-F 2 "" H 5100 2700 50  0001 C CNN
+F 2 "Capacitors_SMD:C_0805" H 5100 2700 50  0001 C CNN
 F 3 "" H 5100 2700 50  0001 C CNN
 	1    5100 2700
@@
 F 0 "C16" V 6250 1700 50  0000 L CNN
 F 1 "10n" V 6500 1700 50  0000 L CNN
-F 2 "" H 6400 1800 50  0001 C CNN
+F 2 "Capacitors_SMD:C_0805" H 6400 1800 50  0001 C CNN
 F 3 "" H 6400 1800 50  0001 C CNN
 	1    6400 1800
@@
 F 0 "R7" V 7300 2350 50  0000 L CNN
 F 1 "5K6 1%" V 7500 2250 50  0000 L CNN
-F 2 "" H 7400 2400 50  0001 C CNN
+F 2 "Resistors_SMD:R_0805" H 7400 2400 50  0001 C CNN
 F 3 "" H 7400 2400 50  0001 C CNN
 	1    7400 2400
@@
 F 0 "R10" V 7300 2650 50  0000 L CNN
 F 1 "1k 1%" V 7500 2650 50  0000 L CNN
-F 2 "" H 7400 2700 50  0001 C CNN
+F 2 "Resistors_SMD:R_0805" H 7400 2700 50  0001 C CNN
 F 3 "" H 7400 2700 50  0001 C CNN
 	1    7400 2700
@@
 F 0 "C7" H 8210 2570 50  0000 L CNN
 F 1 "100u" H 8210 2420 50  0000 L CNN
-F 2 "" H 8200 2500 50  0001 C CNN
+F 2 "Capacitors_SMD:CP_Elec_6.3x5.3" H 8200 2500 50  0001 C CNN
 F 3 "" H 8200 2500 50  0001 C CNN
 	1    8200 2500
@@
 F 0 "C15" H 7860 2570 50  0000 L CNN
 F 1 "100n" H 7860 2420 50  0000 L CNN
-F 2 "" H 7850 2500 50  0001 C CNN
+F 2 "Capacitors_SMD:C_0805" H 7850 2500 50  0001 C CNN
 F 3 "" H 7850 2500 50  0001 C CNN
 	1    7850 2500
@@
 F 0 "C22" H 3160 4920 50  0000 L CNN
 F 1 "100nF" H 3160 4770 50  0000 L CNN
-F 2 "" H 3150 4850 50  0001 C CNN
+F 2 "Capacitors_SMD:C_0805" H 3150 4850 50  0001 C CNN
 F 3 "" H 3150 4850 50  0001 C CNN
 	1    3150 4850
@@
 F 0 "R18" V 2600 4400 50  0000 L CNN
 F 1 "10k" V 2800 4300 50  0000 L CNN
-F 2 "" H 2700 4450 50  0001 C CNN
+F 2 "Resistors_SMD:R_0805" H 2700 4450 50  0001 C CNN
 F 3 "" H 2700 4450 50  0001 C CNN
 	1    2700 4450
@@
 F 0 "R17" V 2600 4800 50  0000 L CNN
 F 1 "10k" V 2800 4700 50  0000 L CNN
-F 2 "" H 2700 4850 50  0001 C CNN
+F 2 "Resistors_SMD:R_0805" H 2700 4850 50  0001 C CNN
 F 3 "" H 2700 4850 50  0001 C CNN
 	1    2700 4850
@@
 F 0 "Q4" V 5500 4550 50  0000 L BNN
 F 1 "FDN340P" V 5500 3900 50  0000 L BNN
-F 2 "SOT23-3" H 5630 4550 20  0001 C CNN
+F 2 "TO_SOT_Packages_SMD:SOT-23" H 5630 4550 20  0001 C CNN
 F 3 "" H 5600 4400 60  0001 C CNN
 	1    5600 4400
@@
 F 0 "R20" V 4800 4500 50  0000 L CNN
 F 1 "10k" V 5000 4400 50  0000 L CNN
-F 2 "" H 4900 4550 50  0001 C CNN
+F 2 "Resistors_SMD:R_0805" H 4900 4550 50  0001 C CNN
 F 3 "" H 4900 4550 50  0001 C CNN
 	1    4900 4550
@@
 F 0 "R16" V 5100 5350 50  0000 L CNN
 F 1 "10k" V 5300 5250 50  0000 L CNN
-F 2 "" H 5200 5400 50  0001 C CNN
+F 2 "Resistors_SMD:R_0805" H 5200 5400 50  0001 C CNN
 F 3 "" H 5200 5400 50  0001 C CNN
 	1    5200 5400
@@
 F 0 "C23" H 4510 4420 50  0000 L CNN
 F 1 "100nF" H 4510 4270 50  0000 L CNN
-F 2 "" H 4500 4350 50  0001 C CNN
+F 2 "Capacitors_SMD:C_0805" H 4500 4350 50  0001 C CNN
 F 3 "" H 4500 4350 50  0001 C CNN
 	1    4500 4350
@@
 F 0 "C24" H 8410 4770 50  0000 L CNN
 F 1 "100nF" H 8410 4620 50  0000 L CNN
-F 2 "" H 8400 4700 50  0001 C CNN
+F 2 "Capacitors_SMD:C_0805" H 8400 4700 50  0001 C CNN
 F 3 "" H 8400 4700 50  0001 C CNN
 	1    8400 4700
