File: Hardware/KiCad/Grape/Microcontroller.sch (KiCad schematic (older format))
At the start: 0 parts

Commit message: Microcontrolador añadido
Parts:
- added C12: 1uF, symbol C_Small
- added C13: 100nF, symbol C_Small
- added C14: 10nF, symbol C_Small
- added C5, C6: 0.1uF, symbol C_Small
- added D2: YELLOW, symbol LED_Small_ALT
- added D4: PURPLE, symbol LED_Small_ALT
- added J?: ARDUINO_R3, ARDUINO_R3, symbol ARDUINO_R3
- added R2, R8: 1k, symbol R_Small
- added R3: 10k, symbol R_Small
- added S2: RESET, TACTILE-PTH, symbol SWITCH-MOMENTARY-2PTH
- added U4: ATMEGA328P_TQFP, TQFP32-08, symbol ATMEGA328P_TQFP
- added Y1: 16MHz, symbol Resonator_Small
Connections:
- net labels added: +5V, AD0, AD1, AD2, AD3, AD4/SDA, AD5/SCL, AD6, AD7, AREF, DTR, GND, IO2/PIN2, IO3/PIN3, IO4/PIN4, IO5/PIN5, IO6/PIN6, IO7/PIN7, IO8/PIN8, IO9/PIN9, MISO/PIN12, MOSI/PIN11, RESET, RX, SCK/PIN13, SS/PIN10, TX
- wire segments 0 -> 102

Commit message: Alimentacion comenzada
Parts:
- gave numbers to parts that had none: 1
Connections:
- net labels added: +3.3V, VIN
- wire segments 102 -> 104
Other:
- moved on the sheet: C12, C13, C14, C5, C6, D2, D4, J3, R2, R3, R8, S2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

Commit message: Alimentacion terminada
Parts:
- renumbered D2 to D3
Changed lines of the file:
@@
 $EndComp
 $Comp
-L LED_Small_ALT D2
+L LED_Small_ALT D3
 U 1 1 5A5C2C40
 P 5300 5150
-F 0 "D2" H 5250 5275 50  0000 L CNN
+F 0 "D3" H 5250 5275 50  0000 L CNN
 F 1 "YELLOW" H 5200 5050 50  0000 L CNN
 F 2 "" V 5300 5150 50  0001 C CNN
@@
 	1700 3750 2750 3750
 $Comp
-L GND #PWR?
+L GND #PWR20
 U 1 1 5A5C2EBD
 P 5050 5250
-F 0 "#PWR?" H 5050 5000 50  0001 C CNN
+F 0 "#PWR20" H 5050 5000 50  0001 C CNN
 F 1 "GND" H 5050 5100 50  0000 C CNN
 F 2 "" H 5050 5250 60  0000 C CNN
@@
 $EndComp
 $Comp
-L GND #PWR?
+L GND #PWR18
 U 1 1 5A5C3052
 P 3100 4950
-F 0 "#PWR?" H 3100 4700 50  0001 C CNN
+F 0 "#PWR18" H 3100 4700 50  0001 C CNN
 F 1 "GND" H 3100 4800 50  0000 C CNN
 F 2 "" H 3100 4950 60  0000 C CNN
@@
 Connection ~ 3100 4850
 $Comp
-L GND #PWR?
+L GND #PWR15
 U 1 1 5A5C30CE
 P 1700 3900
-F 0 "#PWR?" H 1700 3650 50  0001 C CNN
+F 0 "#PWR15" H 1700 3650 50  0001 C CNN
 F 1 "GND" H 1700 3750 50  0000 C CNN
 F 2 "" H 1700 3900 60  0000 C CNN
@@
 AREF
 $Comp
-L +5V #PWR?
+L +5V #PWR19
 U 1 1 5A5C31DF
 P 3150 2150
-F 0 "#PWR?" H 3150 2000 50  0001 C CNN
+F 0 "#PWR19" H 3150 2000 50  0001 C CNN
 F 1 "+5V" H 3150 2290 50  0000 C CNN
 F 2 "" H 3150 2150 60  0000 C CNN
@@
 $EndComp
 $Comp
-L GND #PWR?
+L GND #PWR16
 U 1 1 5A5C3AE5
 P 1800 2750
-F 0 "#PWR?" H 1800 2500 50  0001 C CNN
+F 0 "#PWR16" H 1800 2500 50  0001 C CNN
 F 1 "GND" H 1800 2600 50  0000 C CNN
 F 2 "" H 1800 2750 60  0000 C CNN
@@
 Connection ~ 2950 2650
 $Comp
-L +5V #PWR?
+L +5V #PWR17
 U 1 1 5A5C3C26
 P 2950 2150
-F 0 "#PWR?" H 2950 2000 50  0001 C CNN
+F 0 "#PWR17" H 2950 2000 50  0001 C CNN
 F 1 "+5V" H 2950 2290 50  0000 C CNN
 F 2 "" H 2950 2150 60  0000 C CNN
@@
 Wire Wire Line
 	5150 3150 6050 3150
-Wire Wire Line
-	5150 3250 6050 3250
-Wire Wire Line
-	5150 3350 6050 3350
 Wire Wire Line
 	5150 3550 6050 3550
@@
 $EndComp
 $Comp
-L GND #PWR?
+L GND #PWR25
 U 1 1 5A5C5726
 P 8850 5550
-F 0 "#PWR?" H 8850 5300 50  0001 C CNN
+F 0 "#PWR25" H 8850 5300 50  0001 C CNN
 F 1 "GND" H 8850 5400 50  0000 C CNN
 F 2 "" H 8850 5550 60  0000 C CNN
@@
 Connection ~ 8850 5450
 $Comp
-L +5V #PWR?
+L +5V #PWR24
 U 1 1 5A5C58DC
 P 8850 5000
-F 0 "#PWR?" H 8850 4850 50  0001 C CNN
+F 0 "#PWR24" H 8850 4850 50  0001 C CNN
 F 1 "+5V" H 8850 5140 50  0000 C CNN
 F 2 "" H 8850 5000 60  0000 C CNN
@@
 $EndComp
 $Comp
-L +5V #PWR?
+L +5V #PWR27
 U 1 1 5A5C5FB8
 P 9650 4850
-F 0 "#PWR?" H 9650 4700 50  0001 C CNN
+F 0 "#PWR27" H 9650 4700 50  0001 C CNN
 F 1 "+5V" H 9650 4990 50  0000 C CNN
 F 2 "" H 9650 4850 60  0000 C CNN
@@
 $EndComp
 $Comp
-L GND #PWR?
+L GND #PWR28
 U 1 1 5A5C5FF7
 P 9650 5550
-F 0 "#PWR?" H 9650 5300 50  0001 C CNN
+F 0 "#PWR28" H 9650 5300 50  0001 C CNN
 F 1 "GND" H 9650 5400 50  0000 C CNN
 F 2 "" H 9650 5550 60  0000 C CNN
@@
 Connection ~ 8050 3400
 $Comp
-L GND #PWR?
+L GND #PWR23
 U 1 1 5A5C7818
 P 7950 3600
-F 0 "#PWR?" H 7950 3350 50  0001 C CNN
+F 0 "#PWR23" H 7950 3350 50  0001 C CNN
 F 1 "GND" H 7950 3450 50  0000 C CNN
 F 2 "" H 7950 3600 60  0000 C CNN
@@
 	7950 3400 7950 3600
 $Comp
-L GND #PWR?
+L GND #PWR26
 U 1 1 5A5C78D0
 P 9550 4300
-F 0 "#PWR?" H 9550 4050 50  0001 C CNN
+F 0 "#PWR26" H 9550 4050 50  0001 C CNN
 F 1 "GND" H 9550 4150 50  0000 C CNN
 F 2 "" H 9550 4300 60  0000 C CNN
@@
 $EndComp
 $Comp
-L +5V #PWR?
+L +5V #PWR29
 U 1 1 5A5C7B73
 P 10000 3650
-F 0 "#PWR?" H 10000 3500 50  0001 C CNN
+F 0 "#PWR29" H 10000 3500 50  0001 C CNN
 F 1 "+5V" H 10000 3790 50  0000 C CNN
 F 2 "" H 10000 3650 60  0000 C CNN
@@
 AD5/SCL
 $Comp
-L +5V #PWR?
+L +5V #PWR21
 U 1 1 5A5C8726
 P 7100 2550
-F 0 "#PWR?" H 7100 2400 50  0001 C CNN
+F 0 "#PWR21" H 7100 2400 50  0001 C CNN
 F 1 "+5V" H 7100 2690 50  0000 C CNN
 F 2 "" H 7100 2550 60  0000 C CNN
@@
 $EndComp
 $Comp
-L +3.3V #PWR?
+L +3.3V #PWR22
 U 1 1 5A5C8B00
 P 7350 2550
-F 0 "#PWR?" H 7350 2400 50  0001 C CNN
+F 0 "#PWR22" H 7350 2400 50  0001 C CNN
 F 1 "+3.3V" H 7350 2690 50  0000 C CNN
 F 2 "" H 7350 2550 60  0000 C CNN
@@
 Text GLabel 9550 4100 2    39   Input ~ 0
 RESET
+Wire Wire Line
+	5150 3250 6050 3250
+Wire Wire Line
+	6050 3350 5150 3350
 $EndSCHEMATC

Commit message: Esquema terminado y  ERC pasado
Other:
- note added: "ARDUINO UNO\n HEADERS"
- moved on the sheet: C12, C13, C14, D4, J3, R8

Commit message: cvpcb terminado
Parts:
- C12, C13, C14, C5, C6: footprint (none) -> Capacitors_SMD:C_0603
- D2: renamed from D3; footprint (none) -> LEDs:LED_0603
- D4: footprint (none) -> LEDs:LED_0603
- J3: footprint ARDUINO_R3 -> Boards:UNO_R3_SHIELD_ICSP
- R2, R3, R8: footprint (none) -> Resistors_SMD:R_0805
- S2: footprint TACTILE-PTH -> Buttons_Switches_THT:SW_Tactile_SPST_Angled_PTS645Vx39-2LFS
- U4: footprint TQFP32-08 -> Housings_QFP:TQFP-32_7x7mm_Pitch0.8mm
- Y1: footprint (none) -> Clocks:RESONATOR-SMD-3.2X1.3
Changed lines of the file:
@@
 F 0 "U4" H 3450 5180 50  0000 L BNN
 F 1 "ATMEGA328P_TQFP" H 3450 2550 50  0000 L BNN
-F 2 "TQFP32-08" H 4280 4000 20  0001 C CNN
+F 2 "Housings_QFP:TQFP-32_7x7mm_Pitch0.8mm" H 4280 4000 20  0001 C CNN
 F 3 "" H 4250 3850 60  0001 C CNN
 	1    4250 3850
@@
 F 0 "C5" H 1710 3620 50  0000 L CNN
 F 1 "0.1uF" H 1710 3470 50  0000 L CNN
-F 2 "" H 1700 3550 50  0001 C CNN
+F 2 "Capacitors_SMD:C_0603" H 1700 3550 50  0001 C CNN
 F 3 "" H 1700 3550 50  0001 C CNN
 	1    1700 3550
@@
 $EndComp
 $Comp
-L LED_Small_ALT D3
+L LED_Small_ALT D2
 U 1 1 5A5C2C40
 P 5300 5150
-F 0 "D3" H 5250 5275 50  0000 L CNN
+F 0 "D2" H 5250 5275 50  0000 L CNN
 F 1 "YELLOW" H 5200 5050 50  0000 L CNN
-F 2 "" V 5300 5150 50  0001 C CNN
+F 2 "LEDs:LED_0603" V 5300 5150 50  0001 C CNN
 F 3 "" V 5300 5150 50  0001 C CNN
 	1    5300 5150
@@
 F 0 "R3" H 2980 2470 50  0000 L CNN
 F 1 "10k" H 2980 2410 50  0000 L CNN
-F 2 "" H 2950 2450 50  0001 C CNN
+F 2 "Resistors_SMD:R_0805" H 2950 2450 50  0001 C CNN
 F 3 "" H 2950 2450 50  0001 C CNN
 	1    2950 2450
@@
 F 0 "Y1" V 2750 3700 50  0000 L CNN
 F 1 "16MHz" V 3150 3650 50  0000 L CNN
-F 2 "" H 2925 3750 50  0001 C CNN
+F 2 "Clocks:RESONATOR-SMD-3.2X1.3" H 2925 3750 50  0001 C CNN
 F 3 "" H 2925 3750 50  0001 C CNN
 	1    2950 3750
@@
 F 0 "S2" H 2000 2750 50  0000 L BNN
 F 1 "RESET" H 2000 2550 50  0000 L BNN
-F 2 "TACTILE-PTH" H 2130 2800 20  0001 C CNN
+F 2 "Buttons_Switches_THT:SW_Tactile_SPST_Angled_PTS645Vx39-2LFS" H 2130 2800 20  0001 C CNN
 F 3 "" H 2100 2650 60  0001 C CNN
 	1    2100 2650
@@
 F 0 "C6" H 2410 2520 50  0000 L CNN
 F 1 "0.1uF" H 2410 2370 50  0000 L CNN
-F 2 "" H 2400 2450 50  0001 C CNN
+F 2 "Capacitors_SMD:C_0603" H 2400 2450 50  0001 C CNN
 F 3 "" H 2400 2450 50  0001 C CNN
 	1    2400 2450
@@
 F 0 "R2" V 5550 5100 50  0000 L CNN
 F 1 "1k" V 5750 5100 50  0000 L CNN
-F 2 "" H 5650 5150 50  0001 C CNN
+F 2 "Resistors_SMD:R_0805" H 5650 5150 50  0001 C CNN
 F 3 "" H 5650 5150 50  0001 C CNN
 	1    5650 5150
@@
 F 0 "C14" H 5110 6770 50  0000 L CNN
 F 1 "10nF" H 5110 6620 50  0000 L CNN
-F 2 "" H 5100 6700 50  0001 C CNN
+F 2 "Capacitors_SMD:C_0603" H 5100 6700 50  0001 C CNN
 F 3 "" H 5100 6700 50  0001 C CNN
 	1    5100 6700
@@
 F 0 "C13" H 5410 6770 50  0000 L CNN
 F 1 "100nF" H 5410 6620 50  0000 L CNN
-F 2 "" H 5400 6700 50  0001 C CNN
+F 2 "Capacitors_SMD:C_0603" H 5400 6700 50  0001 C CNN
 F 3 "" H 5400 6700 50  0001 C CNN
 	1    5400 6700
@@
 F 0 "C12" H 5710 6770 50  0000 L CNN
 F 1 "1uF" H 5710 6620 50  0000 L CNN
-F 2 "" H 5700 6700 50  0001 C CNN
+F 2 "Capacitors_SMD:C_0603" H 5700 6700 50  0001 C CNN
 F 3 "" H 5700 6700 50  0001 C CNN
 	1    5700 6700
@@
 F 0 "D4" H 6150 6875 50  0000 L CNN
 F 1 "PURPLE" H 6100 6650 50  0000 L CNN
-F 2 "" V 6200 6750 50  0001 C CNN
+F 2 "LEDs:LED_0603" V 6200 6750 50  0001 C CNN
 F 3 "" V 6200 6750 50  0001 C CNN
 	1    6200 6750
@@
 F 0 "R8" V 6100 6400 50  0000 L CNN
 F 1 "1k" V 6300 6400 50  0000 L CNN
-F 2 "" H 6200 6450 50  0001 C CNN
+F 2 "Resistors_SMD:R_0805" H 6200 6450 50  0001 C CNN
 F 3 "" H 6200 6450 50  0001 C CNN
 	1    6200 6450
@@
 F 0 "J3" H 8320 4580 50  0000 L BNN
 F 1 "ARDUINO_R3" H 8300 2050 50  0000 L BNN
-F 2 "ARDUINO_R3" H 8730 3700 20  0001 C CNN
+F 2 "Boards:UNO_R3_SHIELD_ICSP" H 8730 3700 20  0001 C CNN
 F 3 "" H 8700 3550 60  0001 C CNN
 	1    8700 3550

Commit message: Semiconductores colocados en placa y 3D añadido
Parts:
- J3: footprint Boards:UNO_R3_SHIELD_ICSP -> Boards:ARDUINO_R3
Changed lines of the file:
@@
 F 0 "J3" H 8320 4580 50  0000 L BNN
 F 1 "ARDUINO_R3" H 8300 2050 50  0000 L BNN
-F 2 "Boards:UNO_R3_SHIELD_ICSP" H 8730 3700 20  0001 C CNN
+F 2 "Boards:ARDUINO_R3" H 8730 3700 20  0001 C CNN
 F 3 "" H 8700 3550 60  0001 C CNN
 	1    8700 3550
