File: Hardware/KiCad/Grape/Usb_communication.sch (KiCad schematic (older format))
At the start: 20 parts, among them J1 USB_MICROB, Q1 2N7002PW, U1 FT231XS

Commit message: Esquema terminado y  ERC pasado
Other:
- note added: "USB UART\n"

Commit message: cvpcb terminado
Parts:
- C1, C19, C2, C20, C4: footprint (none) -> Capacitors_SMD:C_0805
- C3: footprint (none) -> Capacitors_Tantalum_SMD:CP_Tantalum_Case-A_EIA-3216-18_Reflow
- F2: footprint (none) -> Resistors_SMD:R_1812
- J1: footprint USB-B-MICRO-SMD_V03 -> Connectors_USB:USB_Micro-B_Molex_47346-0001
- LED1: renamed from D1; footprint (none) -> LEDs:LED_0805
- LED2: renamed from D2; footprint (none) -> LEDs:LED_0805
- Q1: footprint SOT323 -> TO_SOT_Packages_SMD:SOT-323_SC-70
- R1, R12, R13, R14, R15, R4, R5, R6: footprint (none) -> Resistors_SMD:R_0805
- U1: footprint SSOP-20 -> SMD_Packages:SSOP-20
Changed lines of the file:
@@
 F 0 "Q1" V 7850 3700 50  0000 L BNN
 F 1 "2N7002PW" V 8250 3650 50  0000 L BNN
-F 2 "SOT323" H 8080 4000 20  0001 C CNN
+F 2 "TO_SOT_Packages_SMD:SOT-323_SC-70" H 8080 4000 20  0001 C CNN
 F 3 "" H 8050 3850 60  0001 C CNN
 	1    8050 3850
@@
 F 0 "F2" V 3275 3450 50  0000 C CNN
 F 1 "500mA" V 3425 3450 50  0000 C CNN
-F 2 "" H 3400 3250 50  0001 L CNN
+F 2 "Resistors_SMD:R_1812" H 3400 3250 50  0001 L CNN
 F 3 "" H 3350 3450 50  0001 C CNN
 	1    3350 3450
@@
 F 0 "R12" V 3450 3600 50  0000 L CNN
 F 1 "27R" V 3450 3800 50  0000 L CNN
-F 2 "" H 3550 3750 50  0001 C CNN
+F 2 "Resistors_SMD:R_0805" H 3550 3750 50  0001 C CNN
 F 3 "" H 3550 3750 50  0001 C CNN
 	1    3550 3750
@@
 F 0 "C3" H 4560 4370 50  0000 L CNN
 F 1 "CP1_SmalluF" H 4560 4220 50  0000 L CNN
-F 2 "" H 4550 4300 50  0001 C CNN
+F 2 "Capacitors_Tantalum_SMD:CP_Tantalum_Case-A_EIA-3216-18_Reflow" H 4550 4300 50  0001 C CNN
 F 3 "" H 4550 4300 50  0001 C CNN
 	1    4550 4300
@@
 $EndComp
 $Comp
-L LED_Small_ALT D1
+L LED_Small_ALT LED1
 U 1 1 5A5B9670
 P 9100 4250
-F 0 "D1" H 9150 4150 50  0000 L CNN
+F 0 "LED1" H 9150 4150 50  0000 L CNN
 F 1 "RED" H 8900 4150 50  0000 L CNN
-F 2 "" V 9100 4250 50  0001 C CNN
+F 2 "LEDs:LED_0805" V 9100 4250 50  0001 C CNN
 F 3 "" V 9100 4250 50  0001 C CNN
 	1    9100 4250
@@
 F 0 "J1" H 2110 4170 50  0000 L BNN
 F 1 "USB_MICROB" H 2100 3460 50  0000 L BNN
-F 2 "USB-B-MICRO-SMD_V03" H 2330 4000 20  0001 C CNN
+F 2 "Connectors_USB:USB_Micro-B_Molex_47346-0001" H 2330 4000 20  0001 C CNN
 F 3 "" H 2300 3850 60  0000 C CNN
 	1    2300 3850
@@
 F 0 "U1" H 6000 4850 50  0000 L CNN
 F 1 "FT231XS" H 6850 4850 50  0000 L CNN
-F 2 "SSOP-20" H 6550 4050 50  0001 C CNN
+F 2 "SMD_Packages:SSOP-20" H 6550 4050 50  0001 C CNN
 F 3 "" H 6550 4050 50  0001 C CNN
 	1    6550 4050
@@
 F 0 "C4" H 3060 4370 50  0000 L CNN
 F 1 "0.1uF" H 3060 4220 50  0000 L CNN
-F 2 "" H 3050 4300 50  0001 C CNN
+F 2 "Capacitors_SMD:C_0805" H 3050 4300 50  0001 C CNN
 F 3 "" H 3050 4300 50  0001 C CNN
 	1    3050 4300
@@
 F 0 "R13" V 3650 3700 50  0000 L CNN
 F 1 "27R" V 3650 3900 50  0000 L CNN
-F 2 "" H 3550 3850 50  0001 C CNN
+F 2 "Resistors_SMD:R_0805" H 3550 3850 50  0001 C CNN
 F 3 "" H 3550 3850 50  0001 C CNN
 	1    3550 3850
@@
 F 0 "C20" H 3450 4400 50  0000 L CNN
 F 1 "47pF" H 3450 4200 50  0000 L CNN
-F 2 "" H 3650 4300 50  0001 C CNN
+F 2 "Capacitors_SMD:C_0805" H 3650 4300 50  0001 C CNN
 F 3 "" H 3650 4300 50  0001 C CNN
 	1    3650 4300
@@
 F 0 "C19" H 3850 4400 50  0000 L CNN
 F 1 "47pF" H 3850 4200 50  0000 L CNN
-F 2 "" H 3800 4300 50  0001 C CNN
+F 2 "Capacitors_SMD:C_0805" H 3800 4300 50  0001 C CNN
 F 3 "" H 3800 4300 50  0001 C CNN
 	1    3800 4300
@@
 F 0 "C2" H 4160 4370 50  0000 L CNN
 F 1 "0.1uF" H 4160 4220 50  0000 L CNN
-F 2 "" H 4150 4300 50  0001 C CNN
+F 2 "Capacitors_SMD:C_0805" H 4150 4300 50  0001 C CNN
 F 3 "" H 4150 4300 50  0001 C CNN
 	1    4150 4300
@@
 F 0 "C1" H 5610 4370 50  0000 L CNN
 F 1 "0.1uF" H 5610 4220 50  0000 L CNN
-F 2 "" H 5600 4300 50  0001 C CNN
+F 2 "Capacitors_SMD:C_0805" H 5600 4300 50  0001 C CNN
 F 3 "" H 5600 4300 50  0001 C CNN
 	1    5600 4300
@@
 F 0 "R5" V 7850 2700 50  0000 L CNN
 F 1 "1k" V 7850 3000 50  0000 L CNN
-F 2 "" H 7800 2900 50  0001 C CNN
+F 2 "Resistors_SMD:R_0805" H 7800 2900 50  0001 C CNN
 F 3 "" H 7800 2900 50  0001 C CNN
 	1    7800 2900
@@
 F 0 "R6" V 7900 2900 50  0000 L CNN
 F 1 "1k" V 7900 3100 50  0000 L CNN
-F 2 "" H 7800 3050 50  0001 C CNN
+F 2 "Resistors_SMD:R_0805" H 7800 3050 50  0001 C CNN
 F 3 "" H 7800 3050 50  0001 C CNN
 	1    7800 3050
@@
 TX
 $Comp
-L LED_Small_ALT D2
+L LED_Small_ALT LED2
 U 1 1 5A5BC688
 P 9350 4250
-F 0 "D2" H 9400 4150 50  0000 L CNN
+F 0 "LED2" H 9400 4150 50  0000 L CNN
 F 1 "GREEN" H 9100 4150 50  0000 L CNN
-F 2 "" V 9350 4250 50  0001 C CNN
+F 2 "LEDs:LED_0805" V 9350 4250 50  0001 C CNN
 F 3 "" V 9350 4250 50  0001 C CNN
 	1    9350 4250
@@
 F 0 "R4" V 9150 3950 50  0000 L CNN
 F 1 "1k" V 9150 3650 50  0000 L CNN
-F 2 "" H 9100 3850 50  0001 C CNN
+F 2 "Resistors_SMD:R_0805" H 9100 3850 50  0001 C CNN
 F 3 "" H 9100 3850 50  0001 C CNN
 	1    9100 3850
@@
 F 0 "R1" V 9400 3950 50  0000 L CNN
 F 1 "1k" V 9400 3650 50  0000 L CNN
-F 2 "" H 9350 3850 50  0001 C CNN
+F 2 "Resistors_SMD:R_0805" H 9350 3850 50  0001 C CNN
 F 3 "" H 9350 3850 50  0001 C CNN
 	1    9350 3850
@@
 F 0 "R14" V 7900 3450 50  0000 L CNN
 F 1 "10k" V 7900 3650 50  0000 L CNN
-F 2 "" H 7800 3650 50  0001 C CNN
+F 2 "Resistors_SMD:R_0805" H 7800 3650 50  0001 C CNN
 F 3 "" H 7800 3650 50  0001 C CNN
 	1    7800 3650
@@
 F 0 "R15" V 8250 3550 50  0000 L CNN
 F 1 "10k" V 8450 3550 50  0000 L CNN
-F 2 "" H 8350 3650 50  0001 C CNN
+F 2 "Resistors_SMD:R_0805" H 8350 3650 50  0001 C CNN
 F 3 "" H 8350 3650 50  0001 C CNN
 	1    8350 3650

Commit message: Terminada
Parts:
- J1: footprint Connectors_USB:USB_Micro-B_Molex_47346-0001 -> Connectors_USB:USB_Micro-B_Molex-105017-0001
Changed lines of the file:
@@
 F 0 "J1" H 2110 4170 50  0000 L BNN
 F 1 "USB_MICROB" H 2100 3460 50  0000 L BNN
-F 2 "Connectors_USB:USB_Micro-B_Molex_47346-0001" H 2330 4000 20  0001 C CNN
+F 2 "Connectors_USB:USB_Micro-B_Molex-105017-0001" H 2330 4000 20  0001 C CNN
 F 3 "" H 2300 3850 60  0000 C CNN
 	1    2300 3850
