File: Hardware/KiCad/Grape.kicad_pcb (KiCad board)
At the start: 2 copper layers, 68.6 x 53.3 mm, 105 parts, among them J1 USB_MICROB, J19 POWER_JACKPTH, J3 ARDUINO_R3, P1 CONN_01X03, P10 CONN_01X03, P11 CONN_01X03, P12 CONN_01X03, P13 CONN_01X03, P14 CONN_01X03, P15 CONN_01X03, P16 CONN_01X03, P17 CONN_01X03, P18 CONN_01X03, P19 CONN_01X03, P2 CONN_01X03, P20 CONN_01X03, P21 CONN_01X03, P22 CONN_01X03, P23 I2C, P3 CONN_01X03, P4 CONN_01X03, P5 CONN_01X03, P6 CONN_01X03, P7 CONN_01X03, P8 CONN_01X03, P9 CONN_01X03, Q1 2N7002PW, Q4 FDN340P, Q5 FDN340P, SW1 SW_SPDT, U1 FT231XS, U2 LM358, U3 AMS1117-3.3, U4 ATMEGA328P_TQFP, U8 MP2307SO, Y1 16MHz

Commit message: preparando archivos
Other:
- board text added: "OFF - ON"
- board text removed: "ON - OFF"
