File: Hardware/KiCad/_autosave-Usb_communication.sch (KiCad schematic (older format))
At the start: 23 parts, among them P1 CONN_01X03, P10 CONN_01X03, P11 CONN_01X03, P12 CONN_01X03, P13 CONN_01X03, P14 CONN_01X03, P15 CONN_01X03, P16 CONN_01X03, P17 CONN_01X03, P18 CONN_01X03, P19 CONN_01X03, P2 CONN_01X03, P20 CONN_01X03, P21 CONN_01X03, P22 CONN_01X03, P23 I2C, P3 CONN_01X03, P4 CONN_01X03, P5 CONN_01X03, P6 CONN_01X03, P7 CONN_01X03, P8 CONN_01X03, P9 CONN_01X03

Commit message: preparando archivos
Parts:
- removed P1, P10, P11, P12, P13, P14, P15, P16, P17, P18, P19, P2, P20, P21, P22, P3, P4, P5, P6, P7, P8, P9: CONN_01X03, lib_sch:Pin_Header_Straight_1x03_Pitch2.54mm, symbol Grape:CONN_01X03
- removed P23: I2C, lib_sch:JST_PH_S4B-PH-K_04x2.00mm_Angled, symbol Grape:CONN_01X04
- added C1, C2, C4: 100nF, lib_sch:C_0805, symbol Grape:C_Small
- added C19, C20: 47pF, lib_sch:C_0805, symbol Grape:C_Small
- added C3: 10nF, lib_sch:CP_Tantalum_Case-A_EIA-3216-18_Reflow, symbol Grape:CP1_Small
- added F2: 500mA, lib_sch:R_1812, symbol Grape:Polyfuse_Small
- added J1: USB_MICROB, lib_sch:USB_Micro-B_Molex-105017-0001, symbol Grape:USB_MICROB_PLUGCONN-11752
- added LED1: RED, lib_sch:LED_0805, symbol Grape:LED_Small_ALT
- added LED2: GREEN, lib_sch:LED_0805, symbol Grape:LED_Small_ALT
- added Q1: 2N7002PW, lib_sch:SOT-323_SC-70, symbol Grape:MOSFET-NCHANNEL2N7002PW
- added R1, R4, R5, R6: 1k, lib_sch:R_0805, symbol Grape:R_Small
- added R12, R13: 27R, lib_sch:R_0805, symbol Grape:R_Small
- added R14, R15: 10k, lib_sch:R_0805, symbol Grape:R_Small
- added U1: FT231XS, lib_sch:SSOP-20, symbol Grape:FT231XS
- added USB?: HRO-TYPE-C-31-M-12, symbol Type-C:HRO-TYPE-C-31-M-12
Connections:
- net labels added: +3.3V, DTR, USB_5V
- net labels removed: AD0, AD1, AD2, AD3, AD4/SDA, AD5/SCL, AD6, AD7, IO2/PIN2, IO3/PIN3, IO4/PIN4, IO5/PIN5, IO6/PIN6, IO7/PIN7, IO8/PIN8, IO9/PIN9, MISO/PIN12, MOSI/PIN11, SCK/PIN13, SS/PIN10
- wire segments 94 -> 97
- no-connect marks 0 -> 9
Other:
- note added: "USB UART\n"
