File: Hardware/KiCad/Microcontroller.sch (KiCad schematic (older format))
At the start: 14 parts, among them J3 ARDUINO_R3, U4 ATMEGA328P_TQFP, Y1 16MHz

Commit message: Cambiando el árbol de carpetas
Parts:
- C12, C13, C14, C5, C6: footprint Capacitors_SMD:C_0603 -> lib_sch:C_0603
- D2, D4: footprint LEDs:LED_0603 -> lib_sch:LED_0603
- J3: footprint Boards:ARDUINO_R3 -> lib_sch:ARDUINO_R3
- R2, R3, R8: footprint Resistors_SMD:R_0805 -> lib_sch:R_0805
- S2: footprint Buttons_Switches_THT:SW_Tactile_SPST_Angled_PTS645Vx39-2LFS -> lib_sch:SW_Tactile_SPST_Angled_PTS645Vx39-2LFS
- U4: footprint Housings_QFP:TQFP-32_7x7mm_Pitch0.8mm -> lib_sch:TQFP-32_7x7mm_Pitch0.8mm
- Y1: footprint Clocks:RESONATOR-SMD-3.2X1.3 -> lib_sch:RESONATOR-SMD-3.2X1.3
Changed lines of the file:
@@
 F 0 "U4" H 3450 5180 50  0000 L BNN
 F 1 "ATMEGA328P_TQFP" H 3450 2550 50  0000 L BNN
-F 2 "Housings_QFP:TQFP-32_7x7mm_Pitch0.8mm" H 4280 4000 20  0001 C CNN
+F 2 "lib_sch:TQFP-32_7x7mm_Pitch0.8mm" H 4280 4000 20  0001 C CNN
 F 3 "" H 4250 3850 60  0001 C CNN
 	1    4250 3850
@@
 F 0 "C5" H 1710 3620 50  0000 L CNN
 F 1 "0.1uF" H 1710 3470 50  0000 L CNN
-F 2 "Capacitors_SMD:C_0603" H 1700 3550 50  0001 C CNN
+F 2 "lib_sch:C_0603" H 1700 3550 50  0001 C CNN
 F 3 "" H 1700 3550 50  0001 C CNN
 	1    1700 3550
@@
 F 0 "D2" H 5250 5275 50  0000 L CNN
 F 1 "YELLOW" H 5200 5050 50  0000 L CNN
-F 2 "LEDs:LED_0603" V 5300 5150 50  0001 C CNN
+F 2 "lib_sch:LED_0603" V 5300 5150 50  0001 C CNN
 F 3 "" V 5300 5150 50  0001 C CNN
 	1    5300 5150
@@
 F 0 "R3" H 2980 2470 50  0000 L CNN
 F 1 "10k" H 2980 2410 50  0000 L CNN
-F 2 "Resistors_SMD:R_0805" H 2950 2450 50  0001 C CNN
+F 2 "lib_sch:R_0805" H 2950 2450 50  0001 C CNN
 F 3 "" H 2950 2450 50  0001 C CNN
 	1    2950 2450
@@
 F 0 "Y1" V 2750 3700 50  0000 L CNN
 F 1 "16MHz" V 3150 3650 50  0000 L CNN
-F 2 "Clocks:RESONATOR-SMD-3.2X1.3" H 2925 3750 50  0001 C CNN
+F 2 "lib_sch:RESONATOR-SMD-3.2X1.3" H 2925 3750 50  0001 C CNN
 F 3 "" H 2925 3750 50  0001 C CNN
 	1    2950 3750
@@
 F 0 "S2" H 2000 2750 50  0000 L BNN
 F 1 "RESET" H 2000 2550 50  0000 L BNN
-F 2 "Buttons_Switches_THT:SW_Tactile_SPST_Angled_PTS645Vx39-2LFS" H 2130 2800 20  0001 C CNN
+F 2 "lib_sch:SW_Tactile_SPST_Angled_PTS645Vx39-2LFS" H 2130 2800 20  0001 C CNN
 F 3 "" H 2100 2650 60  0001 C CNN
 	1    2100 2650
@@
 F 0 "C6" H 2410 2520 50  0000 L CNN
 F 1 "0.1uF" H 2410 2370 50  0000 L CNN
-F 2 "Capacitors_SMD:C_0603" H 2400 2450 50  0001 C CNN
+F 2 "lib_sch:C_0603" H 2400 2450 50  0001 C CNN
 F 3 "" H 2400 2450 50  0001 C CNN
 	1    2400 2450
@@
 F 0 "R2" V 5550 5100 50  0000 L CNN
 F 1 "1k" V 5750 5100 50  0000 L CNN
-F 2 "Resistors_SMD:R_0805" H 5650 5150 50  0001 C CNN
+F 2 "lib_sch:R_0805" H 5650 5150 50  0001 C CNN
 F 3 "" H 5650 5150 50  0001 C CNN
 	1    5650 5150
@@
 F 0 "C14" H 5110 6770 50  0000 L CNN
 F 1 "10nF" H 5110 6620 50  0000 L CNN
-F 2 "Capacitors_SMD:C_0603" H 5100 6700 50  0001 C CNN
+F 2 "lib_sch:C_0603" H 5100 6700 50  0001 C CNN
 F 3 "" H 5100 6700 50  0001 C CNN
 	1    5100 6700
@@
 F 0 "C13" H 5410 6770 50  0000 L CNN
 F 1 "100nF" H 5410 6620 50  0000 L CNN
-F 2 "Capacitors_SMD:C_0603" H 5400 6700 50  0001 C CNN
+F 2 "lib_sch:C_0603" H 5400 6700 50  0001 C CNN
 F 3 "" H 5400 6700 50  0001 C CNN
 	1    5400 6700
@@
 F 0 "C12" H 5710 6770 50  0000 L CNN
 F 1 "1uF" H 5710 6620 50  0000 L CNN
-F 2 "Capacitors_SMD:C_0603" H 5700 6700 50  0001 C CNN
+F 2 "lib_sch:C_0603" H 5700 6700 50  0001 C CNN
 F 3 "" H 5700 6700 50  0001 C CNN
 	1    5700 6700
@@
 F 0 "D4" H 6150 6875 50  0000 L CNN
 F 1 "PURPLE" H 6100 6650 50  0000 L CNN
-F 2 "LEDs:LED_0603" V 6200 6750 50  0001 C CNN
+F 2 "lib_sch:LED_0603" V 6200 6750 50  0001 C CNN
 F 3 "" V 6200 6750 50  0001 C CNN
 	1    6200 6750
@@
 F 0 "R8" V 6100 6400 50  0000 L CNN
 F 1 "1k" V 6300 6400 50  0000 L CNN
-F 2 "Resistors_SMD:R_0805" H 6200 6450 50  0001 C CNN
+F 2 "lib_sch:R_0805" H 6200 6450 50  0001 C CNN
 F 3 "" H 6200 6450 50  0001 C CNN
 	1    6200 6450
@@
 F 0 "J3" H 8320 4580 50  0000 L BNN
 F 1 "ARDUINO_R3" H 8300 2050 50  0000 L BNN
-F 2 "Boards:ARDUINO_R3" H 8730 3700 20  0001 C CNN
+F 2 "lib_sch:ARDUINO_R3" H 8730 3700 20  0001 C CNN
 F 3 "" H 8700 3550 60  0001 C CNN
 	1    8700 3550

Commit message: Valores cambiados
Parts:
- C5, C6: value 0.1uF -> 100nF

Commit message: preparando archivos
Parts:
- C12, C13, C14, C5, C6: symbol C_Small -> Grape:C_Small
- D2, D4: symbol LED_Small_ALT -> Grape:LED_Small_ALT
- J3: symbol ARDUINO_R3 -> Grape:ARDUINO_R3
- R2, R3, R8: symbol R_Small -> Grape:R_Small
- S2: symbol SWITCH-MOMENTARY-2PTH -> Grape:SWITCH-MOMENTARY-2PTH
- U4: symbol ATMEGA328P_TQFP -> Grape:ATMEGA328P_TQFP
- Y1: symbol Resonator_Small -> Grape:Resonator_Small
Changed lines of the file:
@@
-EESchema Schematic File Version 2
-LIBS:Grape
-EELAYER 25 0
+EESchema Schematic File Version 4
+LIBS:Grape-cache
+EELAYER 26 0
 EELAYER END
 $Descr A4 11693 8268
@@
 $EndDescr
 $Comp
-L ATMEGA328P_TQFP U4
+L Grape:ATMEGA328P_TQFP U4
 U 1 1 5A5C2AAB
 P 4250 3850
@@
 $EndComp
 $Comp
-L C_Small C5
+L Grape:C_Small C5
 U 1 1 5A5C2C21
 P 1700 3550
@@
 $EndComp
 $Comp
-L LED_Small_ALT D2
+L Grape:LED_Small_ALT D2
 U 1 1 5A5C2C40
 P 5300 5150
@@
 $EndComp
 $Comp
-L R_Small R3
+L Grape:R_Small R3
 U 1 1 5A5C2C73
 P 2950 2450
@@
 $EndComp
 $Comp
-L Resonator_Small Y1
+L Grape:Resonator_Small Y1
 U 1 1 5A5C2C9C
 P 2950 3750
@@
 	1700 3750 2750 3750
 $Comp
-L GND #PWR062
+L Grape:GND #PWR062
 U 1 1 5A5C2EBD
 P 5050 5250
@@
 $EndComp
 $Comp
-L GND #PWR063
+L Grape:GND #PWR063
 U 1 1 5A5C3052
 P 3100 4950
@@
 Connection ~ 3100 4850
 $Comp
-L GND #PWR064
+L Grape:GND #PWR064
 U 1 1 5A5C30CE
 P 1700 3900
@@
 AREF
 $Comp
-L +5V #PWR065
+L Grape:+5V #PWR065
 U 1 1 5A5C31DF
 P 3150 2150
@@
 	2300 2650 3250 2650
 $Comp
-L SWITCH-MOMENTARY-2PTH S2
+L Grape:SWITCH-MOMENTARY-2PTH S2
 U 1 1 5A5C32D8
 P 2100 2650
@@
 $EndComp
 $Comp
-L GND #PWR066
+L Grape:GND #PWR066
 U 1 1 5A5C3AE5
 P 1800 2750
@@
 Connection ~ 2950 2650
 $Comp
-L +5V #PWR067
+L Grape:+5V #PWR067
 U 1 1 5A5C3C26
 P 2950 2150
@@
 RESET
 $Comp
-L C_Small C6
+L Grape:C_Small C6
 U 1 1 5A5C3D11
 P 2400 2450
@@
 	5050 5150 5050 5250
 $Comp
-L R_Small R2
+L Grape:R_Small R2
 U 1 1 5A5C4E73
 P 5650 5150
@@
 Connection ~ 5900 4950
 $Comp
-L C_Small C14
+L Grape:C_Small C14
 U 1 1 5A5C52EB
 P 5100 6700
@@
 $EndComp
 $Comp
-L C_Small C13
+L Grape:C_Small C13
 U 1 1 5A5C55A3
 P 5400 6700
@@
 $EndComp
 $Comp
-L C_Small C12
+L Grape:C_Small C12
 U 1 1 5A5C55D9
 P 5700 6700
@@
 $EndComp
 $Comp
-L GND #PWR068
+L Grape:GND #PWR068
 U 1 1 5A5C5726
 P 5400 7000
@@
 Connection ~ 5400 6900
 $Comp
-L +5V #PWR069
+L Grape:+5V #PWR069
 U 1 1 5A5C58DC
 P 5400 6450
@@
 	5700 6500 5700 6600
 $Comp
-L LED_Small_ALT D4
+L Grape:LED_Small_ALT D4
 U 1 1 5A5C5C11
 P 6200 6750
@@
 $EndComp
 $Comp
-L R_Small R8
+L Grape:R_Small R8
 U 1 1 5A5C5DC5
 P 6200 6450
@@
 $EndComp
 $Comp
-L +5V #PWR070
+L Grape:+5V #PWR070
 U 1 1 5A5C5FB8
 P 6200 6300
@@
 $EndComp
 $Comp
-L GND #PWR071
+L Grape:GND #PWR071
 U 1 1 5A5C5FF7
 P 6200 7000
@@
 	6200 6350 6200 6300
 $Comp
-L ARDUINO_R3 J3
+L Grape:ARDUINO_R3 J3
 U 1 1 5A5C633B
 P 8700 3550
@@
 Connection ~ 8050 4050
 $Comp
-L GND #PWR072
+L Grape:GND #PWR072
 U 1 1 5A5C7818
 P 7950 4250
@@
 	7950 4050 7950 4250
 $Comp
-L GND #PWR073
+L Grape:GND #PWR073
 U 1 1 5A5C78D0
 P 9550 4950
@@
 $EndComp
 $Comp
-L +5V #PWR074
+L Grape:+5V #PWR074
 U 1 1 5A5C7B73
 P 10000 4300
@@
 AD5/SCL
 $Comp
-L +5V #PWR075
+L Grape:+5V #PWR075
 U 1 1 5A5C8726
 P 7100 3200
@@
 $EndComp
 $Comp
-L +3.3V #PWR076
+L Grape:+3.3V #PWR076
 U 1 1 5A5C8B00
 P 7350 3200
@@
 $Bitmap
 Pos 10850 6250
-Scale 0,950000
+Scale 0.000000
 Data
 89 50 4E 47 0D 0A 1A 0A 00 00 00 0D 49 48 44 52 00 00 00 C1 00 00 00 8F 08 06 00 00 00 43 10 BF
@@
 $Bitmap
 Pos 7250 6700
-Scale 0,950000
+Scale 0.000000
 Data
 89 50 4E 47 0D 0A 1A 0A 00 00 00 0D 49 48 44 52 00 00 00 91 00 00 00 36 08 06 00 00 00 C7 C1 7B

Commit message: Esquema terminado
Falta comprobar
Parts:
- added JP?: Jumper_NC_Dual, symbol device:Jumper_NC_Dual
- D2: value YELLOW -> BLUE
Connections:
- net +3V3: now also JP?.3
- net +5V: now also JP?.1; no longer C12.1, C13.1, C14.1, J3.VCC, R3.1, R8.2, U4.18 (AVCC), U4.4 (VCC), U4.6 (VCC)
- new net VCC: C12.1, C13.1, C14.1, J3.VCC, JP?.2, R3.1, R8.2, U4.18 (AVCC), U4.4 (VCC), U4.6 (VCC)
Changed lines of the file:
@@
 P 5300 5150
 F 0 "D2" H 5250 5275 50  0000 L CNN
-F 1 "YELLOW" H 5200 5050 50  0000 L CNN
+F 1 "BLUE" H 5200 5050 50  0000 L CNN
 F 2 "lib_sch:LED_0603" V 5300 5150 50  0001 C CNN
 F 3 "" V 5300 5150 50  0001 C CNN
@@
 $EndComp
 Wire Wire Line
-	3100 4650 3100 4950
+	3100 4650 3100 4750
 Wire Wire Line
 	3100 4650 3250 4650
@@
 $EndComp
 Wire Wire Line
-	1700 3650 1700 3900
+	1700 3650 1700 3750
 Connection ~ 1700 3750
 Wire Wire Line
 	1700 3450 1700 3250
 Wire Wire Line
-	1400 3250 3250 3250
+	1400 3250 1700 3250
 Connection ~ 1700 3250
 Text GLabel 1400 3250 0    39   Input ~ 0
 AREF
-$Comp
-L Grape:+5V #PWR065
-U 1 1 5A5C31DF
-P 3150 2150
-F 0 "#PWR065" H 3150 2000 50  0001 C CNN
-F 1 "+5V" H 3150 2290 50  0000 C CNN
-F 2 "" H 3150 2150 60  0000 C CNN
-F 3 "" H 3150 2150 60  0000 C CNN
-	1    3150 2150
-	1    0    0    -1
-$EndComp
 Wire Wire Line
 	3150 3050 3250 3050
 Wire Wire Line
-	3150 2150 3150 3050
+	3150 2150 3150 2850
 Wire Wire Line
 	3250 2850 3150 2850
@@
 Connection ~ 3150 2950
 Wire Wire Line
-	2300 2650 3250 2650
+	2300 2650 2400 2650
 $Comp
 L Grape:SWITCH-MOMENTARY-2PTH S2
@@
 	2950 2550 2950 2650
 Connection ~ 2950 2650
-$Comp
-L Grape:+5V #PWR067
-U 1 1 5A5C3C26
-P 2950 2150
-F 0 "#PWR067" H 2950 2000 50  0001 C CNN
-F 1 "+5V" H 2950 2290 50  0000 C CNN
-F 2 "" H 2950 2150 60  0000 C CNN
-F 3 "" H 2950 2150 60  0000 C CNN
-	1    2950 2150
-	1    0    0    -1
-$EndComp
 Wire Wire Line
 	2950 2150 2950 2350
@@
 	5150 4850 6050 4850
 Wire Wire Line
-	5150 4950 6050 4950
+	5150 4950 5900 4950
 Text GLabel 6050 2650 2    39   Input ~ 0
 AD0
@@
 	5100 6800 5100 6900
 Wire Wire Line
-	5100 6900 5700 6900
-Wire Wire Line
-	5400 6800 5400 7000
+	5100 6900 5400 6900
+Wire Wire Line
+	5400 6800 5400 6900
 Wire Wire Line
 	5700 6900 5700 6800
 Connection ~ 5400 6900
-$Comp
-L Grape:+5V #PWR069
-U 1 1 5A5C58DC
-P 5400 6450
-F 0 "#PWR069" H 5400 6300 50  0001 C CNN
-F 1 "+5V" H 5400 6590 50  0000 C CNN
-F 2 "" H 5400 6450 60  0000 C CNN
-F 3 "" H 5400 6450 60  0000 C CNN
-	1    5400 6450
-	1    0    0    -1
-$EndComp
 Wire Wire Line
 	5100 6600 5100 6500
 Wire Wire Line
-	5100 6500 5700 6500
-Wire Wire Line
-	5400 6450 5400 6600
+	5100 6500 5400 6500
+Wire Wire Line
+	5400 6450 5400 6500
 Connection ~ 5400 6500
 Wire Wire Line
@@
 $EndComp
 $Comp
-L Grape:+5V #PWR070
-U 1 1 5A5C5FB8
-P 6200 6300
-F 0 "#PWR070" H 6200 6150 50  0001 C CNN
-F 1 "+5V" H 6200 6440 50  0000 C CNN
-F 2 "" H 6200 6300 60  0000 C CNN
-F 3 "" H 6200 6300 60  0000 C CNN
-	1    6200 6300
-	1    0    0    -1
-$EndComp
-$Comp
 L Grape:GND #PWR071
 U 1 1 5A5C5FF7
@@
 	8200 3950 8050 3950
 Wire Wire Line
-	8050 3950 8050 4150
+	8050 3950 8050 4050
 Wire Wire Line
 	8050 4150 8200 4150
 Wire Wire Line
-	7950 4050 8200 4050
+	7950 4050 8050 4050
 Connection ~ 8050 4050
 $Comp
@@
 F 3 "" H 9550 4950 60  0000 C CNN
 	1    9550 4950
-	1    0    0    -1
-$EndComp
-$Comp
-L Grape:+5V #PWR074
-U 1 1 5A5C7B73
-P 10000 4300
-F 0 "#PWR074" H 10000 4150 50  0001 C CNN
-F 1 "+5V" H 10000 4440 50  0000 C CNN
-F 2 "" H 10000 4300 60  0000 C CNN
-F 3 "" H 10000 4300 60  0000 C CNN
-	1    10000 4300
 	1    0    0    -1
 $EndComp
@@
 	7350 3750 7350 3200
 Wire Wire Line
-	7100 3200 7100 3650
+	7100 3200 7100 3350
 Connection ~ 7100 3350
 Text GLabel 9550 4450 2    39   Input ~ 0
@@
 Text Notes 6950 2550 0    59   ~ 0
 ARDUINO UNO\n HEADERS
+Wire Wire Line
+	3100 4750 3100 4850
+Wire Wire Line
+	3100 4850 3100 4950
+Wire Wire Line
+	1700 3750 1700 3900
+Wire Wire Line
+	1700 3250 3250 3250
+Wire Wire Line
+	3150 2850 3150 2950
+Wire Wire Line
+	3150 2950 3150 3050
+Wire Wire Line
+	2950 2650 3250 2650
+Wire Wire Line
+	2550 2650 2950 2650
+Wire Wire Line
+	2400 2650 2550 2650
+Wire Wire Line
+	5900 4950 6050 4950
+Wire Wire Line
+	5400 6900 5700 6900
+Wire Wire Line
+	5400 6900 5400 7000
+Wire Wire Line
+	5400 6500 5700 6500
+Wire Wire Line
+	5400 6500 5400 6600
+Wire Wire Line
+	8050 4050 8050 4150
+Wire Wire Line
+	8050 4050 8200 4050
+Wire Wire Line
+	7100 3350 7100 3650
+$Comp
+L power:VCC #PWR?
+U 1 1 5FD65448
+P 3150 2150
+F 0 "#PWR?" H 3150 2000 50  0001 C CNN
+F 1 "VCC" H 3167 2323 50  0000 C CNN
+F 2 "" H 3150 2150 50  0001 C CNN
+F 3 "" H 3150 2150 50  0001 C CNN
+	1    3150 2150
+	1    0    0    -1
+$EndComp
+$Comp
+L power:VCC #PWR?
+U 1 1 5FD66883
+P 2950 2150
+F 0 "#PWR?" H 2950 2000 50  0001 C CNN
+F 1 "VCC" H 2967 2323 50  0000 C CNN
+F 2 "" H 2950 2150 50  0001 C CNN
+F 3 "" H 2950 2150 50  0001 C CNN
+	1    2950 2150
+	1    0    0    -1
+$EndComp
+$Comp
+L power:VCC #PWR?
+U 1 1 5FD66AB2
+P 6200 6300
+F 0 "#PWR?" H 6200 6150 50  0001 C CNN
+F 1 "VCC" H 6217 6473 50  0000 C CNN
+F 2 "" H 6200 6300 50  0001 C CNN
+F 3 "" H 6200 6300 50  0001 C CNN
+	1    6200 6300
+	1    0    0    -1
+$EndComp
+$Comp
+L power:VCC #PWR?
+U 1 1 5FD693E6
+P 5400 6450
+F 0 "#PWR?" H 5400 6300 50  0001 C CNN
+F 1 "VCC" H 5417 6623 50  0000 C CNN
+F 2 "" H 5400 6450 50  0001 C CNN
+F 3 "" H 5400 6450 50  0001 C CNN
+	1    5400 6450
+	1    0    0    -1
+$EndComp
+$Comp
+L power:VCC #PWR?
+U 1 1 5FD6EAF5
+P 10000 4300
+F 0 "#PWR?" H 10000 4150 50  0001 C CNN
+F 1 "VCC" H 10017 4473 50  0000 C CNN
+F 2 "" H 10000 4300 50  0001 C CNN
+F 3 "" H 10000 4300 50  0001 C CNN
+	1    10000 4300
+	1    0    0    -1
+$EndComp
+$Comp
+L device:Jumper_NC_Dual JP?
+U 1 1 5FD71B80
+P 4150 6250
+F 0 "JP?" H 4150 6489 50  0000 C CNN
+F 1 "Jumper_NC_Dual" H 4150 6398 50  0000 C CNN
+F 2 "" H 4150 6250 50  0001 C CNN
+F 3 "" H 4150 6250 50  0001 C CNN
+	1    4150 6250
+	1    0    0    -1
+$EndComp
+$Comp
+L power:VCC #PWR?
+U 1 1 5FD73F68
+P 4150 6400
+F 0 "#PWR?" H 4150 6250 50  0001 C CNN
+F 1 "VCC" H 4168 6573 50  0000 C CNN
+F 2 "" H 4150 6400 50  0001 C CNN
+F 3 "" H 4150 6400 50  0001 C CNN
+	1    4150 6400
+	-1   0    0    1
+$EndComp
+Wire Wire Line
+	4150 6350 4150 6400
+$Comp
+L Grape:+3.3V #PWR?
+U 1 1 5FD79FFB
+P 4600 6200
+F 0 "#PWR?" H 4600 6050 50  0001 C CNN
+F 1 "+3.3V" H 4600 6340 50  0000 C CNN
+F 2 "" H 4600 6200 60  0000 C CNN
+F 3 "" H 4600 6200 60  0000 C CNN
+	1    4600 6200
+	1    0    0    -1
+$EndComp
+Wire Wire Line
+	4400 6250 4600 6250
+Wire Wire Line
+	4600 6250 4600 6200
+$Comp
+L Grape:+5V #PWR?
+U 1 1 5FD80CC5
+P 3700 6200
+F 0 "#PWR?" H 3700 6050 50  0001 C CNN
+F 1 "+5V" H 3700 6340 50  0000 C CNN
+F 2 "" H 3700 6200 60  0000 C CNN
+F 3 "" H 3700 6200 60  0000 C CNN
+	1    3700 6200
+	1    0    0    -1
+$EndComp
+Wire Wire Line
+	3700 6200 3700 6250
+Wire Wire Line
+	3700 6250 3900 6250
 $EndSCHEMATC
